File: pcb/cheating-calc.kicad_sch (KiCad schematic)
At the start: 8 parts, among them J1 Conn_01x04, Q1 MMBF170, Q2 MMBF170, U1 MOUDLE-SEEEDUINO-XIAO-ESP32C3

Commit message: updated the wole project
Other:
- company: (none) -> from SVA
- title: (none) -> esp32-CALC
