File: pcb/cheating-calc.kicad_pcb (KiCad board)
At the start: 2 copper layers, 72 x 22 mm, 8 parts, among them J1 Conn_01x04, Q1 MMBF170, Q2 MMBF170, U1 MOUDLE-SEEEDUINO-XIAO-ESP32C3

Commit message: updated the wole project
Other:
- board size 72 x 22 mm -> 71.5 x 21.7 mm
- board text added: "pitiee9"
- board text removed: "TI-32 v0.1 ChromaLock 2024"

Commit message: updated the readme
Routing:
- net GND: track 0.00 -> 91.3 mm
Changed lines of the file:
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@@
 			(drillshape 0)
 			(scaleselection 1)
-			(outputdirectory "")
+			(outputdirectory "gerber files/")
 		)
 	)
@@
 			)
 		)
-		(property "Datasheet" ""
+		(property "Datasheet" "https://www.diodes.com/assets/Datasheets/ds30104.pdf"
 			(at 0 0 180)
 			(layer "F.Fab")
@@
 			)
 		)
-		(property "Description" "0.5A Id, 60V Vds, N-Channel MOSFET, SOT-23"
+		(property "Description" ""
 			(at 0 0 180)
 			(layer "F.Fab")
@@
 			)
 		)
+		(property ki_fp_filters "SOT?23*")
+		(sheetname "/")
 		(sheetfile "cheating-calc.kicad_sch")
 		(attr smd)
@@
 			)
 		)
-		(property "Datasheet" ""
+		(property "Datasheet" "~"
 			(at 0 0 270)
 			(layer "F.Fab")
@@
 			)
 		)
-		(property "Description" "Generic connector, single row, 01x04, script generated (kicad-library-utils/schlib/autogen/connector/)"
+		(property "Description" ""
 			(at 0 0 270)
 			(layer "F.Fab")
@@
 			)
 		)
+		(property ki_fp_filters "Connector*:*_1x??_*")
+		(sheetname "/")
 		(sheetfile "cheating-calc.kicad_sch")
 		(attr through_hole)
@@
 			)
 		)
-		(property "Datasheet" ""
+		(property "Datasheet" "~"
 			(at 0 0 270)
 			(layer "F.Fab")
@@
 			)
 		)
-		(property "Description" "Resistor"
+		(property "Description" ""
 			(at 0 0 270)
 			(layer "F.Fab")
@@
 			)
 		)
+		(property ki_fp_filters "R_*")
+		(sheetname "/")
 		(sheetfile "cheating-calc.kicad_sch")
 		(attr through_hole)
@@
 			)
 		)
-		(property "Datasheet" ""
+		(property "Datasheet" "~"
 			(at 0 0 270)
 			(layer "F.Fab")
@@
 			)
 		)
-		(property "Description" "Resistor"
+		(property "Description" ""
 			(at 0 0 270)
 			(layer "F.Fab")
@@
 			)
 		)
+		(property ki_fp_filters "R_*")
+		(sheetname "/")
 		(sheetfile "cheating-calc.kicad_sch")
 		(attr through_hole)
@@
 			)
 		)
+		(sheetname "/")
 		(sheetfile "cheating-calc.kicad_sch")
 		(attr through_hole)
@@
 			)
 		)
-		(property "Datasheet" ""
+		(property "Datasheet" "~"
 			(at 0 0 270)
 			(layer "F.Fab")
@@
 			)
 		)
-		(property "Description" "Resistor"
+		(property "Description" ""
 			(at 0 0 270)
 			(layer "F.Fab")
@@
 			)
 		)
+		(property ki_fp_filters "R_*")
+		(sheetname "/")
 		(sheetfile "cheating-calc.kicad_sch")
 		(attr through_hole)
@@
 			)
 		)
-		(property "Datasheet" ""
+		(property "Datasheet" "https://www.diodes.com/assets/Datasheets/ds30104.pdf"
 			(at 0 0 180)
 			(layer "F.Fab")
@@
 			)
 		)
-		(property "Description" "0.5A Id, 60V Vds, N-Channel MOSFET, SOT-23"
+		(property "Description" ""
 			(at 0 0 180)
 			(layer "F.Fab")
@@
 			)
 		)
+		(property ki_fp_filters "SOT?23*")
+		(sheetname "/")
 		(sheetfile "cheating-calc.kicad_sch")
 		(attr smd)
@@
 			)
 		)
-		(property "Datasheet" ""
+		(property "Datasheet" "~"
 			(at 0 0 270)
 			(layer "F.Fab")
@@
 			)
 		)
-		(property "Description" "Resistor"
+		(property "Description" ""
 			(at 0 0 270)
 			(layer "F.Fab")
@@
 			)
 		)
+		(property ki_fp_filters "R_*")
+		(sheetname "/")
 		(sheetfile "cheating-calc.kicad_sch")
 		(attr through_hole)
@@
 		(net 6)
 	)
+	(segment
+		(start 155.488 70.03554)
+		(end 152.52354 73)
+		(width 0.25)
+		(layer "F.Cu")
+		(net 7)
+	)
+	(segment
+		(start 152.84554 52.889)
+		(end 155.488 55.53146)
+		(width 0.25)
+		(layer "F.Cu")
+		(net 7)
+	)
+	(segment
+		(start 136.71446 52.889)
+		(end 152.84554 52.889)
+		(width 0.25)
+		(layer "F.Cu")
+		(net 7)
+	)
+	(segment
+		(start 96.012 70.425919)
+		(end 109.847919 56.59)
+		(width 0.25)
+		(layer "F.Cu")
+		(net 7)
+	)
+	(segment
+		(start 109.847919 56.59)
+		(end 133.01346 56.59)
+		(width 0.25)
+		(layer "F.Cu")
+		(net 7)
+	)
+	(segment
+		(start 155.488 55.53146)
+		(end 155.488 70.03554)
+		(width 0.25)
+		(layer "F.Cu")
+		(net 7)
+	)
+	(segment
+		(start 152.52354 73)
+		(end 151.994 73)
+		(width 0.25)
+		(layer "F.Cu")
+		(net 7)
+	)
+	(segment
+		(start 133.01346 56.59)
+		(end 136.71446 52.889)
+		(width 0.25)
+		(layer "F.Cu")
+		(net 7)
+	)
+	(segment
+		(start 96.012 71.628)
+		(end 96.012 70.425919)
+		(width 0.25)
+		(layer "F.Cu")
+		(net 7)
+	)
+	(segment
+		(start 151.994 73)
+		(end 149.86 70.866)
+		(width 0.25)
+		(layer "F.Cu")
+		(net 7)
+	)
 	(zone
